Commit message: fix(bringup, control, description): fix the structure to work with moveit package

File: src/so101_follower_description/urdf/arm_on_table.urdf.xacro (robot description, xacro)
@@ -1,5 +1,12 @@
 <?xml version='1.0' encoding='utf-8'?>
-<robot name="so_arm" xmlns:xacro="http://www.ros.org/wiki/xacro">
+<robot name="so101_follower" xmlns:xacro="http://www.ros.org/wiki/xacro">
     <xacro:arg name="sim_mode" default="gazebo" />
+    <xacro:arg name="moveit_status" default="false" />
+    <link name="world"/>
+    <joint name="world_to_table" type="fixed">
+        <parent link="world"/>
+        <child  link="table_link"/>
+        <origin xyz="0 0 0.5" rpy="0 0 0"/>
+    </joint>
     <link name="table_link">
         <!-- Inertial block is required for physics -->
@@ -33,6 +40,3 @@
     </joint>
     <xacro:include filename="$(find so101_follower_description)/urdf/so101_follower_with_ros2_control.urdf.xacro" />
-    <xacro:include filename="$(find so101_follower_description)/urdf/so101_follower_with_ros2_control.urdf.xacro">
-        <xacro:arg name="sim_mode" value="${sim_mode}" />
-    </xacro:include>
 </robot>

File: src/so101_follower_description/urdf/robots/so101_follower.urdf.xacro (robot description, xacro)
@@ -3,11 +3,4 @@
 <!-- Onshape https://cad.onshape.com/documents/7715cc284bb430fe6dab4ffd/w/4fd0791b683777b02f8d975a/e/826c553ede3b7592eb9ca800 -->
 <robot name="so101_follower" xmlns:xacro="http://www.ros.org/wiki/xacro">
-  <!-- World Link -->
-  <link name="world"/>
-  <joint name="world_to_base" type="fixed">
-    <parent link="world"/>
-    <child link="base_link"/>
-    <origin xyz="0 0 0" rpy="0 0 0"/>
-  </joint>
   <!-- Materials -->
   <material name="3d_printed">

File: src/so101_follower_description/urdf/so101_follower_with_ros2_control.urdf.xacro (robot description, xacro)
@@ -1,10 +1,14 @@
 <?xml version='1.0' encoding='utf-8'?>
 <robot name="so101_follower" xmlns:xacro="http://www.ros.org/wiki/xacro">
-    <xacro:arg name="sim_mode" default="gazebo" />
-    <!-- ros2 control and sensors for simulated robot in gazebo ignition -->
-    <xacro:if value="${'$(arg sim_mode)' == 'gazebo'}">
-        <xacro:include filename="$(find so101_follower_description)/urdf/ros2_control/sim_gazebo_so101_follower_ros2_control.urdf" />
-    </xacro:if>
-    <xacro:if value="${'$(arg sim_mode)' == 'isaacsim'}">
+    <xacro:arg name="moveit_status" default="false" />
+    <xacro:arg name="sim_mode" default="gazebo" />''
+    <!-- include if moveit_status is false  -->
+    <xacro:if value="${'$(arg moveit_status)' == 'false'}">
+        <!-- ros2 control and sensors for simulated robot in gazebo ignition -->
+        <xacro:if value="${'$(arg sim_mode)' == 'gazebo'}">
+            <xacro:include filename="$(find so101_follower_description)/urdf/ros2_control/sim_gazebo_so101_follower_ros2_control.urdf" />
+        </xacro:if>
+        <xacro:if value="${'$(arg sim_mode)' == 'isaacsim'}">
+        </xacro:if>
     </xacro:if>
     <xacro:if value="${'$(arg sim_mode)' == 'real_robot'}">
