Commit message: chore: so101_follower_description name change to so101_description

File: src/so101_description/urdf/apriltag_markers/apriltag.urdf.xacro (robot description, xacro)
@@ -1,5 +1,5 @@
                 <?xml version='1.0' encoding='utf-8'?>
 <robot name="apriltags" xmlns:xacro="http://www.ros.org/wiki/xacro">
-    <xacro:include filename="$(find so101_follower_description)/urdf/apriltag_marker.xacro" />
+    <xacro:include filename="$(find so101_description)/urdf/apriltag_marker.xacro" />
     <link name="world"/>
     <joint name="world_to_base" type="fixed">

File: src/so101_description/urdf/arm_on_table.urdf.xacro (robot description, xacro)
@@ -39,4 +39,4 @@
         <origin xyz="0 0.4 0.47" rpy="0 0 0"/>
     </joint>
-    <xacro:include filename="$(find so101_follower_description)/urdf/so101_follower_with_ros2_control.urdf.xacro" />
+    <xacro:include filename="$(find so101_description)/urdf/so101_follower_with_ros2_control.urdf.xacro" />
 </robot>

File: src/so101_description/urdf/robots/so101_follower.urdf.xacro (robot description, xacro)
@@ -22,5 +22,5 @@
       <origin xyz="0.0206915 0.0221255 0.0300817" rpy="1.5708 -1.23909e-16 2.33147e-15"/>
       <geometry>
-        <mesh filename="package://so101_follower_description/meshes/base_motor_holder_so101_v1.stl"/>
+        <mesh filename="package://so101_description/meshes/base_motor_holder_so101_v1.stl"/>
       </geometry>
       <material name="3d_printed"/>
@@ -29,5 +29,5 @@
       <origin xyz="0.0206915 0.0221255 0.0300817" rpy="1.5708 -1.23909e-16 2.33147e-15"/>
       <geometry>
-        <mesh filename="package://so101_follower_description/meshes/base_motor_holder_so101_v1.stl"/>
+        <mesh filename="package://so101_description/meshes/base_motor_holder_so101_v1.stl"/>
       </geometry>
     </collision>
@@ -36,5 +36,5 @@
       <origin xyz="0.0207909 0.0221255 0.0300817" rpy="1.5708 -0 0"/>
       <geometry>
-        <mesh filename="package://so101_follower_description/meshes/base_so101_v2.stl"/>
+        <mesh filename="package://so101_description/meshes/base_so101_v2.stl"/>
       </geometry>
       <material name="3d_printed"/>
@@ -43,5 +43,5 @@
       <origin xyz="0.0207909 0.0221255 0.0300817" rpy="1.5708 -0 0"/>
       <geometry>
-        <mesh filename="package://so101_follower_description/meshes/base_so101_v2.stl"/>
+        <mesh filename="package://so101_description/meshes/base_so101_v2.stl"/>
       </geometry>
     </collision>
@@ -50,5 +50,5 @@
       <origin xyz="0.0207909 -0.0105745 0.0761817" rpy="-2.20282e-15 2.77556e-17 -1.5708"/>
       <geometry>
-        <mesh filename="package://so101_follower_description/meshes/sts3215_03a_v1.stl"/>
+        <mesh filename="package://so101_description/meshes/sts3215_03a_v1.stl"/>
       </geometry>
       <material name="sts3215"/>
@@ -57,5 +57,5 @@
       <origin xyz="0.0207909 -0.0105745 0.0761817" rpy="-2.20282e-15 2.77556e-17 -1.5708"/>
       <geometry>
-        <mesh filename="package://so101_follower_description/meshes/sts3215_03a_v1.stl"/>
+        <mesh filename="package://so101_description/meshes/sts3215_03a_v1.stl"/>
       </geometry>
     </collision>
@@ -64,5 +64,5 @@
       <origin xyz="0.0205915 0.0467435 0.0798817" rpy="1.5708 -1.21716e-14 2.33147e-15"/>
       <geometry>
-        <mesh filename="package://so101_follower_description/meshes/waveshare_mounting_plate_so101_v2.stl"/>
+        <mesh filename="package://so101_description/meshes/waveshare_mounting_plate_so101_v2.stl"/>
       </geometry>
       <material name="3d_printed"/>
@@ -71,5 +71,5 @@
       <origin xyz="0.0205915 0.0467435 0.0798817" rpy="1.5708 -1.21716e-14 2.33147e-15"/>
       <geometry>
-        <mesh filename="package://so101_follower_description/meshes/waveshare_mounting_plate_so101_v2.stl"/>
+        <mesh filename="package://so101_description/meshes/waveshare_mounting_plate_so101_v2.stl"/>
       </geometry>
     </collision>
@@ -86,5 +86,5 @@
       <origin xyz="-0.0303992 0.000422241 -0.0417" rpy="1.5708 1.5708 0"/>
       <geometry>
-        <mesh filename="package://so101_follower_description/meshes/sts3215_03a_v1.stl"/>
+        <mesh filename="package://so101_description/meshes/sts3215_03a_v1.stl"/>
       </geometry>
       <material name="sts3215"/>
@@ -93,5 +93,5 @@
       <origin xyz="-0.0303992 0.000422241 -0.0417" rpy="1.5708 1.5708 0"/>
       <geometry>
-        <mesh filename="package://so101_follower_description/meshes/sts3215_03a_v1.stl"/>
+        <mesh filename="package://so101_description/meshes/sts3215_03a_v1.stl"/>
       </geometry>
     </collision>
@@ -100,5 +100,5 @@
       <origin xyz="-0.0675992 -0.000177759 0.0158499" rpy="1.5708 -1.5708 0"/>
       <geometry>
-        <mesh filename="package://so101_follower_description/meshes/motor_holder_so101_base_v1.stl"/>
+        <mesh filename="package://so101_description/meshes/motor_holder_so101_base_v1.stl"/>
       </geometry>
       <material name="3d_printed"/>
@@ -107,5 +107,5 @@
       <origin xyz="-0.0675992 -0.000177759 0.0158499" rpy="1.5708 -1.5708 0"/>
       <geometry>
-        <mesh filename="package://so101_follower_description/meshes/motor_holder_so101_base_v1.stl"/>
+        <mesh filename="package://so101_description/meshes/motor_holder_so101_base_v1.stl"/>
       </geometry>
     </collision>
@@ -114,5 +114,5 @@
       <origin xyz="0.0122008 2.22413e-05 0.0464" rpy="-1.5708 -0 0"/>
       <geometry>
-        <mesh filename="package://so101_follower_description/meshes/rotation_pitch_so101_v1.stl"/>
+        <mesh filename="package://so101_description/meshes/rotation_pitch_so101_v1.stl"/>
       </geometry>
       <material name="3d_printed"/>
@@ -121,5 +121,5 @@
       <origin xyz="0.0122008 2.22413e-05 0.0464" rpy="-1.5708 -0 0"/>
       <geometry>
-        <mesh filename="package://so101_follower_description/meshes/rotation_pitch_so101_v1.stl"/>
+        <mesh filename="package://so101_description/meshes/rotation_pitch_so101_v1.stl"/>
       </geometry>
     </collision>
@@ -136,5 +136,5 @@
       <origin xyz="-0.11257 -0.0155 0.0187" rpy="-3.14159 -6.8695e-16 -1.5708"/>
       <geometry>
-        <mesh filename="package://so101_follower_description/meshes/sts3215_03a_v1.stl"/>
+        <mesh filename="package://so101_description/meshes/sts3215_03a_v1.stl"/>
       </geometry>
       <material name="sts3215"/>
@@ -143,5 +143,5 @@
       <origin xyz="-0.11257 -0.0155 0.0187" rpy="-3.14159 -6.8695e-16 -1.5708"/>
       <geometry>
-        <mesh filename="package://so101_follower_description/meshes/sts3215_03a_v1.stl"/>
+        <mesh filename="package://so101_description/meshes/sts3215_03a_v1.stl"/>
       </geometry>
     </collision>
@@ -150,5 +150,5 @@
       <origin xyz="-0.065085 0.012 0.0182" rpy="3.14159 -9.35612e-32 0"/>
       <geometry>
-        <mesh filename="package://so101_follower_description/meshes/upper_arm_so101_v1.stl"/>
+        <mesh filename="package://so101_description/meshes/upper_arm_so101_v1.stl"/>
       </geometry>
       <material name="3d_printed"/>
@@ -157,5 +157,5 @@
       <origin xyz="-0.065085 0.012 0.0182" rpy="3.14159 -9.35612e-32 0"/>
       <geometry>
-        <mesh filename="package://so101_follower_description/meshes/upper_arm_so101_v1.stl"/>
+        <mesh filename="package://so101_description/meshes/upper_arm_so101_v1.stl"/>
       </geometry>
     </collision>
@@ -172,5 +172,5 @@
       <origin xyz="-0.0648499 -0.032 0.0182" rpy="-3.14159 -0 3.9443e-31"/>
       <geometry>
-        <mesh filename="package://so101_follower_description/meshes/under_arm_so101_v1.stl"/>
+        <mesh filename="package://so101_description/meshes/under_arm_so101_v1.stl"/>
       </geometry>
       <material name="3d_printed"/>
@@ -179,5 +179,5 @@
       <origin xyz="-0.0648499 -0.032 0.0182" rpy="-3.14159 -0 3.9443e-31"/>
       <geometry>
-        <mesh filename="package://so101_follower_description/meshes/under_arm_so101_v1.stl"/>
+        <mesh filename="package://so101_description/meshes/under_arm_so101_v1.stl"/>
       </geometry>
     </collision>
@@ -186,5 +186,5 @@
       <origin xyz="-0.0648499 -0.032 0.018" rpy="-3.14159 4.73317e-30 7.88861e-31"/>
       <geometry>
-        <mesh filename="package://so101_follower_description/meshes/motor_holder_so101_wrist_v1.stl"/>
+        <mesh filename="package://so101_description/meshes/motor_holder_so101_wrist_v1.stl"/>
       </geometry>
       <material name="3d_printed"/>
@@ -193,5 +193,5 @@
       <origin xyz="-0.0648499 -0.032 0.018" rpy="-3.14159 4.73317e-30 7.88861e-31"/>
       <geometry>
-        <mesh filename="package://so101_follower_description/meshes/motor_holder_so101_wrist_v1.stl"/>
+        <mesh filename="package://so101_description/meshes/motor_holder_so101_wrist_v1.stl"/>
       </geometry>
     </collision>
@@ -200,5 +200,5 @@
       <origin xyz="-0.1224 0.0052 0.0187" rpy="-3.14159 -3.58047e-15 -3.14159"/>
       <geometry>
-        <mesh filename="package://so101_follower_description/meshes/sts3215_03a_v1.stl"/>
+        <mesh filename="package://so101_description/meshes/sts3215_03a_v1.stl"/>
       </geometry>
       <material name="sts3215"/>
@@ -207,5 +207,5 @@
       <origin xyz="-0.1224 0.0052 0.0187" rpy="-3.14159 -3.58047e-15 -3.14159"/>
       <geometry>
-        <mesh filename="package://so101_follower_description/meshes/sts3215_03a_v1.stl"/>
+        <mesh filename="package://so101_description/meshes/sts3215_03a_v1.stl"/>
       </geometry>
     </collision>
@@ -222,5 +222,5 @@
       <origin xyz="5.55112e-17 -0.0424 0.0306" rpy="1.5708 1.5708 0"/>
       <geometry>
-        <mesh filename="package://so101_follower_description/meshes/sts3215_03a_no_horn_v1.stl"/>
+        <mesh filename="package://so101_description/meshes/sts3215_03a_no_horn_v1.stl"/>
       </geometry>
       <material name="sts3215"/>
@@ -229,5 +229,5 @@
       <origin xyz="5.55112e-17 -0.0424 0.0306" rpy="1.5708 1.5708 0"/>
       <geometry>
-        <mesh filename="package://so101_follower_description/meshes/sts3215_03a_no_horn_v1.stl"/>
+        <mesh filename="package://so101_description/meshes/sts3215_03a_no_horn_v1.stl"/>
       </geometry>
     </collision>
@@ -236,5 +236,5 @@
       <origin xyz="0 -0.028 0.0181" rpy="-1.5708 -1.5708 0"/>
       <geometry>
-        <mesh filename="package://so101_follower_description/meshes/wrist_roll_pitch_so101_v2.stl"/>
+        <mesh filename="package://so101_description/meshes/wrist_roll_pitch_so101_v2.stl"/>
       </geometry>
       <material name="3d_printed"/>
@@ -243,5 +243,5 @@
       <origin xyz="0 -0.028 0.0181" rpy="-1.5708 -1.5708 0"/>
       <geometry>
-        <mesh filename="package://so101_follower_description/meshes/wrist_roll_pitch_so101_v2.stl"/>
+        <mesh filename="package://so101_description/meshes/wrist_roll_pitch_so101_v2.stl"/>
       </geometry>
     </collision>
@@ -258,5 +258,5 @@
       <origin xyz="0.0077 0.0001 -0.0234" rpy="-1.5708 -5.55112e-17 -1.38213e-14"/>
       <geometry>
-        <mesh filename="package://so101_follower_description/meshes/sts3215_03a_v1.stl"/>
+        <mesh filename="package://so101_description/meshes/sts3215_03a_v1.stl"/>
       </geometry>
       <material name="sts3215"/>
@@ -265,5 +265,5 @@
       <origin xyz="0.0077 0.0001 -0.0234" rpy="-1.5708 -5.55112e-17 -1.38213e-14"/>
       <geometry>
-        <mesh filename="package://so101_follower_description/meshes/sts3215_03a_v1.stl"/>
+        <mesh filename="package://so101_description/meshes/sts3215_03a_v1.stl"/>
       </geometry>
     </collision>
@@ -272,5 +272,5 @@
       <origin xyz="5.55112e-17 -0.000218214 0.000949706" rpy="-3.14159 -5.55112e-17 -9.17912e-24"/>
       <geometry>
-        <mesh filename="package://so101_follower_description/meshes/wrist_roll_follower_so101_v1_nocamera.stl"/>
+        <mesh filename="package://so101_description/meshes/wrist_roll_follower_so101_v1_nocamera.stl"/>
       </geometry>
       <material name="3d_printed"/>
@@ -279,5 +279,5 @@
       <origin xyz="5.55112e-17 -0.000218214 0.000949706" rpy="-3.14159 -5.55112e-17 -9.17912e-24"/>
       <geometry>
-        <mesh filename="package://so101_follower_description/meshes/wrist_roll_follower_so101_v1_nocamera.stl" />
+        <mesh filename="package://so101_description/meshes/wrist_roll_follower_so101_v1_nocamera.stl" />
       </geometry>
     </collision>
@@ -294,5 +294,5 @@
       <origin xyz="-5.55112e-17 -1.94746e-17 0.0189" rpy="9.53145e-17 -4.66093e-24 0"/>
       <geometry>
-        <mesh filename="package://so101_follower_description/meshes/moving_jaw_so101_v1.stl"/>
+        <mesh filename="package://so101_description/meshes/moving_jaw_so101_v1.stl"/>
       </geometry>
       <material name="3d_printed"/>
@@ -301,5 +301,5 @@
       <origin xyz="-5.55112e-17 -1.94746e-17 0.0189" rpy="9.53145e-17 -4.66093e-24 0"/>
       <geometry>
-        <mesh filename="package://so101_follower_description/meshes/moving_jaw_so101_v1.stl"/>
+        <mesh filename="package://so101_description/meshes/moving_jaw_so101_v1.stl"/>
       </geometry>
     </collision>

File: src/so101_description/urdf/so101_follower_with_ros2_control.urdf.xacro (robot description, xacro)
@@ -7,13 +7,14 @@
         <!-- ros2 control and sensors for simulated robot in gazebo ignition -->
         <xacro:if value="${'$(arg sim_mode)' == 'gazebo'}">
-            <xacro:include filename="$(find so101_follower_description)/urdf/ros2_control/sim_gazebo_so101_follower_ros2_control.urdf" />
+            <xacro:include filename="$(find so101_description)/urdf/ros2_control/sim_gazebo_so101_follower_ros2_control.urdf" />
         </xacro:if>
         <xacro:if value="${'$(arg sim_mode)' == 'isaacsim'}">
+            <xacro:include filename="$(find so101_description)/urdf/ros2_control/sim_isaacsim_so101_follower_ros2_control.urdf" />
         </xacro:if>
         <xacro:if value="${'$(arg sim_mode)' == 'real_robot'}">
-            <xacro:include filename="$(find so101_follower_description)/urdf/ros2_control/real_so101_follower_ros2_control.urdf" />
+            <xacro:include filename="$(find so101_description)/urdf/ros2_control/real_so101_follower_ros2_control.urdf" />
         </xacro:if>
     </xacro:if>
     <!-- robot description -->
-    <xacro:include filename="$(find so101_follower_description)/urdf/robots/so101_follower.urdf.xacro" />
+    <xacro:include filename="$(find so101_description)/urdf/robots/so101_follower.urdf.xacro" />
 </robot>

File: src/so101_moveit_config/config/so101_follower.urdf.xacro (robot description, xacro)
@@ -3,5 +3,5 @@
     <xacro:arg name="initial_positions_file" default="initial_positions.yaml" />
     <!-- Import so101_follower urdf file -->
-    <xacro:include filename="$(find so101_follower_description)/urdf/arm_on_table.urdf.xacro" />
+    <xacro:include filename="$(find so101_description)/urdf/arm_on_table.urdf.xacro" />
     <!-- Import control_xacro -->
     <xacro:include filename="so101_follower.ros2_control.xacro" />
