Commit message: refactor: add prefix to the link name to solve the tf_prefix problem

File: src/so101_description/urdf/robots/so101_arm.urdf.xacro (robot description, xacro)
@@ -2,5 +2,9 @@
 <!-- Generated using onshape-to-robot -->
 <!-- Onshape https://cad.onshape.com/documents/7715cc284bb430fe6dab4ffd/w/4fd0791b683777b02f8d975a/e/826c553ede3b7592eb9ca800 -->
-<robot name="so101_follower" xmlns:xacro="http://www.ros.org/wiki/xacro">
+<!-- Link names are prefixed by arm_prefix (e.g. "follower_" or "leader_") so both arms can
+     share the global TF tree without collision.
+     Joint names (shoulder_pan, etc.) are NOT prefixed — ros2_control uses them plain. -->
+<robot name="so101_arm" xmlns:xacro="http://www.ros.org/wiki/xacro">
+  <xacro:arg name="arm_prefix" default="follower"/>
   <!-- Materials -->
   <material name="3d_printed">
@@ -10,7 +14,6 @@
     <color rgba="0.1 0.1 0.1 1.0"/>
   </material>
-  <!-- Hard-coded calibrated limits (matching your calibration file) -->
   <!-- Link base -->
-  <link name="base_link">
+  <link name="$(arg arm_prefix)_base_link">
     <inertial>
       <origin xyz="0.020739 0.00204287 0.065966" rpy="0 0 0"/>
@@ -18,63 +21,43 @@
       <inertia ixx="0.000136117" ixy="4.59787e-07" ixz="9.75275e-08" iyy="0.000114686" iyz="-4.97151e-06" izz="0.000130364"/>
     </inertial>
-    <!-- Part base_motor_holder_so101_v1 -->
     <visual>
       <origin xyz="0.0206915 0.0221255 0.0300817" rpy="1.5708 -1.23909e-16 2.33147e-15"/>
-      <geometry>
-        <mesh filename="package://so101_description/meshes/base_motor_holder_so101_v1.stl"/>
-      </geometry>
+      <geometry><mesh filename="package://so101_description/meshes/base_motor_holder_so101_v1.stl"/></geometry>
       <material name="3d_printed"/>
     </visual>
     <collision>
       <origin xyz="0.0206915 0.0221255 0.0300817" rpy="1.5708 -1.23909e-16 2.33147e-15"/>
-      <geometry>
-        <mesh filename="package://so101_description/meshes/base_motor_holder_so101_v1.stl"/>
-      </geometry>
-    </collision>
-    <!-- Part base_so101_v2 -->
+      <geometry><mesh filename="package://so101_description/meshes/base_motor_holder_so101_v1.stl"/></geometry>
+    </collision>
     <visual>
       <origin xyz="0.0207909 0.0221255 0.0300817" rpy="1.5708 -0 0"/>
-      <geometry>
-        <mesh filename="package://so101_description/meshes/base_so101_v2.stl"/>
-      </geometry>
+      <geometry><mesh filename="package://so101_description/meshes/base_so101_v2.stl"/></geometry>
       <material name="3d_printed"/>
     </visual>
     <collision>
       <origin xyz="0.0207909 0.0221255 0.0300817" rpy="1.5708 -0 0"/>
-      <geometry>
-        <mesh filename="package://so101_description/meshes/base_so101_v2.stl"/>
-      </geometry>
-    </collision>
-    <!-- Part sts3215_03a_v1 -->
+      <geometry><mesh filename="package://so101_description/meshes/base_so101_v2.stl"/></geometry>
+    </collision>
     <visual>
       <origin xyz="0.0207909 -0.0105745 0.0761817" rpy="-2.20282e-15 2.77556e-17 -1.5708"/>
-      <geometry>
-        <mesh filename="package://so101_description/meshes/sts3215_03a_v1.stl"/>
-      </geometry>
+      <geometry><mesh filename="package://so101_description/meshes/sts3215_03a_v1.stl"/></geometry>
       <material name="sts3215"/>
     </visual>
     <collision>
       <origin xyz="0.0207909 -0.0105745 0.0761817" rpy="-2.20282e-15 2.77556e-17 -1.5708"/>
-      <geometry>
-        <mesh filename="package://so101_description/meshes/sts3215_03a_v1.stl"/>
-      </geometry>
-    </collision>
-    <!-- Part waveshare_mounting_plate_so101_v2 -->
+      <geometry><mesh filename="package://so101_description/meshes/sts3215_03a_v1.stl"/></geometry>
+    </collision>
     <visual>
       <origin xyz="0.0205915 0.0467435 0.0798817" rpy="1.5708 -1.21716e-14 2.33147e-15"/>
-      <geometry>
-        <mesh filename="package://so101_description/meshes/waveshare_mounting_plate_so101_v2.stl"/>
-      </geometry>
+      <geometry><mesh filename="package://so101_description/meshes/waveshare_mounting_plate_so101_v2.stl"/></geometry>
       <material name="3d_printed"/>
     </visual>
     <collision>
       <origin xyz="0.0205915 0.0467435 0.0798817" rpy="1.5708 -1.21716e-14 2.33147e-15"/>
-      <geometry>
-        <mesh filename="package://so101_description/meshes/waveshare_mounting_plate_so101_v2.stl"/>
-      </geometry>
+      <geometry><mesh filename="package://so101_description/meshes/waveshare_mounting_plate_so101_v2.stl"/></geometry>
     </collision>
   </link>
   <!-- Link shoulder -->
-  <link name="shoulder_link">
+  <link name="$(arg arm_prefix)_shoulder_link">
     <inertial>
       <origin xyz="-0.0307604 -1.66727e-05 -0.0252713" rpy="0 0 0"/>
@@ -82,49 +65,34 @@
       <inertia ixx="8.3759e-05" ixy="7.55525e-08" ixz="-1.16342e-06" iyy="8.10403e-05" iyz="1.54663e-07" izz="2.39783e-05"/>
     </inertial>
-    <!-- Part sts3215_03a_v1_2 -->
     <visual>
       <origin xyz="-0.0303992 0.000422241 -0.0417" rpy="1.5708 1.5708 0"/>
-      <geometry>
-        <mesh filename="package://so101_description/meshes/sts3215_03a_v1.stl"/>
-      </geometry>
+      <geometry><mesh filename="package://so101_description/meshes/sts3215_03a_v1.stl"/></geometry>
       <material name="sts3215"/>
     </visual>
     <collision>
       <origin xyz="-0.0303992 0.000422241 -0.0417" rpy="1.5708 1.5708 0"/>
-      <geometry>
-        <mesh filename="package://so101_description/meshes/sts3215_03a_v1.stl"/>
-      </geometry>
-    </collision>
-    <!-- Part motor_holder_so101_base_v1 -->
+      <geometry><mesh filename="package://so101_description/meshes/sts3215_03a_v1.stl"/></geometry>
+    </collision>
     <visual>
       <origin xyz="-0.0675992 -0.000177759 0.0158499" rpy="1.5708 -1.5708 0"/>
-      <geometry>
-        <mesh filename="package://so101_description/meshes/motor_holder_so101_base_v1.stl"/>
-      </geometry>
+      <geometry><mesh filename="package://so101_description/meshes/motor_holder_so101_base_v1.stl"/></geometry>
       <material name="3d_printed"/>
     </visual>
     <collision>
       <origin xyz="-0.0675992 -0.000177759 0.0158499" rpy="1.5708 -1.5708 0"/>
-      <geometry>
-        <mesh filename="package://so101_description/meshes/motor_holder_so101_base_v1.stl"/>
-      </geometry>
-    </collision>
-    <!-- Part rotation_pitch_so101_v1 -->
+      <geometry><mesh filename="package://so101_description/meshes/motor_holder_so101_base_v1.stl"/></geometry>
+    </collision>
     <visual>
       <origin xyz="0.0122008 2.22413e-05 0.0464" rpy="-1.5708 -0 0"/>
-      <geometry>
-        <mesh filename="package://so101_description/meshes/rotation_pitch_so101_v1.stl"/>
-      </geometry>
+      <geometry><mesh filename="package://so101_description/meshes/rotation_pitch_so101_v1.stl"/></geometry>
       <material name="3d_printed"/>
     </visual>
     <collision>
       <origin xyz="0.0122008 2.22413e-05 0.0464" rpy="-1.5708 -0 0"/>
-      <geometry>
-        <mesh filename="package://so101_description/meshes/rotation_pitch_so101_v1.stl"/>
-      </geometry>
+      <geometry><mesh filename="package://so101_description/meshes/rotation_pitch_so101_v1.stl"/></geometry>
     </collision>
   </link>
   <!-- Link upper_arm -->
-  <link name="upper_arm_link">
+  <link name="$(arg arm_prefix)_upper_arm_link">
     <inertial>
       <origin xyz="-0.0898471 -0.00838224 0.0184089" rpy="0 0 0"/>
@@ -132,35 +100,25 @@
       <inertia ixx="4.08002e-05" ixy="-1.97819e-05" ixz="-4.03016e-08" iyy="0.000147318" iyz="8.97326e-09" izz="0.000142487"/>
     </inertial>
-    <!-- Part sts3215_03a_v1_3 -->
     <visual>
       <origin xyz="-0.11257 -0.0155 0.0187" rpy="-3.14159 -6.8695e-16 -1.5708"/>
-      <geometry>
-        <mesh filename="package://so101_description/meshes/sts3215_03a_v1.stl"/>
-      </geometry>
+      <geometry><mesh filename="package://so101_description/meshes/sts3215_03a_v1.stl"/></geometry>
       <material name="sts3215"/>
     </visual>
     <collision>
       <origin xyz="-0.11257 -0.0155 0.0187" rpy="-3.14159 -6.8695e-16 -1.5708"/>
-      <geometry>
-        <mesh filename="package://so101_description/meshes/sts3215_03a_v1.stl"/>
-      </geometry>
-    </collision>
-    <!-- Part upper_arm_so101_v1 -->
+      <geometry><mesh filename="package://so101_description/meshes/sts3215_03a_v1.stl"/></geometry>
+    </collision>
     <visual>
       <origin xyz="-0.065085 0.012 0.0182" rpy="3.14159 -9.35612e-32 0"/>
-      <geometry>
-        <mesh filename="package://so101_description/meshes/upper_arm_so101_v1.stl"/>
-      </geometry>
+      <geometry><mesh filename="package://so101_description/meshes/upper_arm_so101_v1.stl"/></geometry>
       <material name="3d_printed"/>
     </visual>
     <collision>
       <origin xyz="-0.065085 0.012 0.0182" rpy="3.14159 -9.35612e-32 0"/>
-      <geometry>
-        <mesh filename="package://so101_description/meshes/upper_arm_so101_v1.stl"/>
-      </geometry>
+      <geometry><mesh filename="package://so101_description/meshes/upper_arm_so101_v1.stl"/></geometry>
     </collision>
   </link>
   <!-- Link lower_arm -->
-  <link name="lower_arm_link">
+  <link name="$(arg arm_prefix)_lower_arm_link">
     <inertial>
       <origin xyz="-0.0980701 0.00324376 0.0182831" rpy="0 0 0"/>
@@ -168,49 +126,34 @@
       <inertia ixx="2.87438e-05" ixy="7.41152e-06" ixz="1.26409e-06" iyy="0.000159844" iyz="-4.90188e-08" izz="0.00014529"/>
     </inertial>
-    <!-- Part under_arm_so101_v1 -->
     <visual>
       <origin xyz="-0.0648499 -0.032 0.0182" rpy="-3.14159 -0 3.9443e-31"/>
-      <geometry>
-        <mesh filename="package://so101_description/meshes/under_arm_so101_v1.stl"/>
-      </geometry>
+      <geometry><mesh filename="package://so101_description/meshes/under_arm_so101_v1.stl"/></geometry>
       <material name="3d_printed"/>
     </visual>
     <collision>
       <origin xyz="-0.0648499 -0.032 0.0182" rpy="-3.14159 -0 3.9443e-31"/>
-      <geometry>
-        <mesh filename="package://so101_description/meshes/under_arm_so101_v1.stl"/>
-      </geometry>
-    </collision>
-    <!-- Part motor_holder_so101_wrist_v1 -->
+      <geometry><mesh filename="package://so101_description/meshes/under_arm_so101_v1.stl"/></geometry>
+    </collision>
     <visual>
       <origin xyz="-0.0648499 -0.032 0.018" rpy="-3.14159 4.73317e-30 7.88861e-31"/>
-      <geometry>
-        <mesh filename="package://so101_description/meshes/motor_holder_so101_wrist_v1.stl"/>
-      </geometry>
+      <geometry><mesh filename="package://so101_description/meshes/motor_holder_so101_wrist_v1.stl"/></geometry>
       <material name="3d_printed"/>
     </visual>
     <collision>
       <origin xyz="-0.0648499 -0.032 0.018" rpy="-3.14159 4.73317e-30 7.88861e-31"/>
-      <geometry>
-        <mesh filename="package://so101_description/meshes/motor_holder_so101_wrist_v1.stl"/>
-      </geometry>
-    </collision>
-    <!-- Part sts3215_03a_v1_4 -->
+      <geometry><mesh filename="package://so101_description/meshes/motor_holder_so101_wrist_v1.stl"/></geometry>
+    </collision>
     <visual>
       <origin xyz="-0.1224 0.0052 0.0187" rpy="-3.14159 -3.58047e-15 -3.14159"/>
-      <geometry>
-        <mesh filename="package://so101_description/meshes/sts3215_03a_v1.stl"/>
-      </geometry>
+      <geometry><mesh filename="package://so101_description/meshes/sts3215_03a_v1.stl"/></geometry>
       <material name="sts3215"/>
     </visual>
     <collision>
       <origin xyz="-0.1224 0.0052 0.0187" rpy="-3.14159 -3.58047e-15 -3.14159"/>
-      <geometry>
-        <mesh filename="package://so101_description/meshes/sts3215_03a_v1.stl"/>
-      </geometry>
+      <geometry><mesh filename="package://so101_description/meshes/sts3215_03a_v1.stl"/></geometry>
     </collision>
   </link>
   <!-- Link wrist -->
-  <link name="wrist_link">
+  <link name="$(arg arm_prefix)_wrist_link">
     <inertial>
       <origin xyz="-0.000103312 -0.0386143 0.0281156" rpy="0 0 0"/>
@@ -218,35 +161,25 @@
       <inertia ixx="3.68263e-05" ixy="1.7893e-08" ixz="-5.28128e-08" iyy="2.5391e-05" iyz="3.6412e-06" izz="2.1e-05"/>
     </inertial>
-    <!-- Part sts3215_03a_no_horn_v1 -->
     <visual>
       <origin xyz="5.55112e-17 -0.0424 0.0306" rpy="1.5708 1.5708 0"/>
-      <geometry>
-        <mesh filename="package://so101_description/meshes/sts3215_03a_no_horn_v1.stl"/>
-      </geometry>
+      <geometry><mesh filename="package://so101_description/meshes/sts3215_03a_no_horn_v1.stl"/></geometry>
       <material name="sts3215"/>
     </visual>
     <collision>
       <origin xyz="5.55112e-17 -0.0424 0.0306" rpy="1.5708 1.5708 0"/>
-      <geometry>
-        <mesh filename="package://so101_description/meshes/sts3215_03a_no_horn_v1.stl"/>
-      </geometry>
-    </collision>
-    <!-- Part wrist_roll_pitch_so101_v2 -->
+      <geometry><mesh filename="package://so101_description/meshes/sts3215_03a_no_horn_v1.stl"/></geometry>
+    </collision>
     <visual>
       <origin xyz="0 -0.028 0.0181" rpy="-1.5708 -1.5708 0"/>
-      <geometry>
-        <mesh filename="package://so101_description/meshes/wrist_roll_pitch_so101_v2.stl"/>
-      </geometry>
+      <geometry><mesh filename="package://so101_description/meshes/wrist_roll_pitch_so101_v2.stl"/></geometry>
       <material name="3d_printed"/>
     </visual>
     <collision>
       <origin xyz="0 -0.028 0.0181" rpy="-1.5708 -1.5708 0"/>
-      <geometry>
-        <mesh filename="package://so101_description/meshes/wrist_roll_pitch_so101_v2.stl"/>
-      </geometry>
+      <geometry><mesh filename="package://so101_description/meshes/wrist_roll_pitch_so101_v2.stl"/></geometry>
     </collision>
   </link>
   <!-- Link gripper -->
-  <link name="gripper_link">
+  <link name="$(arg arm_prefix)_gripper_link">
     <inertial>
       <origin xyz="0.000213627 0.000245138 -0.025187" rpy="0 0 0"/>
@@ -254,35 +187,25 @@
       <inertia ixx="2.75087e-05" ixy="-3.35241e-07" ixz="-5.7352e-06" iyy="4.33657e-05" iyz="-5.17847e-08" izz="3.45059e-05"/>
     </inertial>
-    <!-- Part sts3215_03a_v1_5 -->
     <visual>
       <origin xyz="0.0077 0.0001 -0.0234" rpy="-1.5708 -5.55112e-17 -1.38213e-14"/>
-      <geometry>
-        <mesh filename="package://so101_description/meshes/sts3215_03a_v1.stl"/>
-      </geometry>
+      <geometry><mesh filename="package://so101_description/meshes/sts3215_03a_v1.stl"/></geometry>
       <material name="sts3215"/>
     </visual>
     <collision>
       <origin xyz="0.0077 0.0001 -0.0234" rpy="-1.5708 -5.55112e-17 -1.38213e-14"/>
-      <geometry>
-        <mesh filename="package://so101_description/meshes/sts3215_03a_v1.stl"/>
-      </geometry>
-    </collision>
-    <!-- Part wrist_roll_follower_so101_v1 -->
+      <geometry><mesh filename="package://so101_description/meshes/sts3215_03a_v1.stl"/></geometry>
+    </collision>
     <visual>
       <origin xyz="5.55112e-17 -0.000218214 0.000949706" rpy="-3.14159 -5.55112e-17 -9.17912e-24"/>
-      <geometry>
-        <mesh filename="package://so101_description/meshes/wrist_roll_follower_so101_v1_nocamera.stl"/>
-      </geometry>
+      <geometry><mesh filename="package://so101_description/meshes/wrist_roll_follower_so101_v1_nocamera.stl"/></geometry>
       <material name="3d_printed"/>
     </visual>
     <collision>
       <origin xyz="5.55112e-17 -0.000218214 0.000949706" rpy="-3.14159 -5.55112e-17 -9.17912e-24"/>
-      <geometry>
-        <mesh filename="package://so101_description/meshes/wrist_roll_follower_so101_v1_nocamera.stl" />
-      </geometry>
+      <geometry><mesh filename="package://so101_description/meshes/wrist_roll_follower_so101_v1_nocamera.stl"/></geometry>
     </collision>
   </link>
   <!-- Link jaw -->
-  <link name="jaw_link">
+  <link name="$(arg arm_prefix)_jaw_link">
     <inertial>
       <origin xyz="-0.00157495 -0.0300244 0.0192755" rpy="0 0 0"/>
@@ -290,132 +213,86 @@
       <inertia ixx="6.61427e-06" ixy="-3.19807e-07" ixz="-5.90717e-09" iyy="1.89032e-06" iyz="-1.09945e-07" izz="5.28738e-06"/>
     </inertial>
-    <!-- Part moving_jaw_so101_v1 -->
     <visual>
       <origin xyz="-5.55112e-17 -1.94746e-17 0.0189" rpy="9.53145e-17 -4.66093e-24 0"/>
-      <geometry>
-        <mesh filename="package://so101_description/meshes/moving_jaw_so101_v1.stl"/>
-      </geometry>
+      <geometry><mesh filename="package://so101_description/meshes/moving_jaw_so101_v1.stl"/></geometry>
       <material name="3d_printed"/>
     </visual>
     <collision>
       <origin xyz="-5.55112e-17 -1.94746e-17 0.0189" rpy="9.53145e-17 -4.66093e-24 0"/>
-      <geometry>
-        <mesh filename="package://so101_description/meshes/moving_jaw_so101_v1.stl"/>
-      </geometry>
-    </collision>
-  </link>
-  <!-- Joint from gripper to jaw -->
+      <geometry><mesh filename="package://so101_description/meshes/moving_jaw_so101_v1.stl"/></geometry>
+    </collision>
+  </link>
+  <!-- Joints (names unchanged — ros2_control uses plain joint names) -->
+  <joint name="shoulder_pan" type="revolute">
+    <origin xyz="0.0207909 -0.0230745 0.0948817" rpy="-3.14159 6.03684e-16 1.5708"/>
+    <parent link="$(arg arm_prefix)_base_link"/>
+    <child link="$(arg arm_prefix)_shoulder_link"/>
+    <axis xyz="0 0 1"/>
+    <limit effort="10" velocity="10" lower="-2.055" upper="2.058"/>
+  </joint>
+  <transmission name="shoulder_pan_trans">
+    <type>transmission_interface/SimpleTransmission</type>
+    <joint name="shoulder_pan"><hardwareInterface>hardware_interface/PositionJointInterface</hardwareInterface></joint>
+    <actuator name="motor1"><hardwareInterface>hardware_interface/PositionJointInterface</hardwareInterface><mechanicalReduction>1</mechanicalReduction></actuator>
+  </transmission>
+  <joint name="shoulder_lift" type="revolute">
+    <origin xyz="-0.0303992 -0.0182778 -0.0542" rpy="-1.5708 -1.5708 0"/>
+    <parent link="$(arg arm_prefix)_shoulder_link"/>
+    <child link="$(arg arm_prefix)_upper_arm_link"/>
+    <axis xyz="0 0 1"/>
+    <limit effort="10" velocity="10" lower="-2.018" upper="2.018"/>
+  </joint>
+  <transmission name="shoulder_lift_trans">
+    <type>transmission_interface/SimpleTransmission</type>
+    <joint name="shoulder_lift"><hardwareInterface>hardware_interface/PositionJointInterface</hardwareInterface></joint>
+    <actuator name="motor2"><hardwareInterface>hardware_interface/PositionJointInterface</hardwareInterface><mechanicalReduction>1</mechanicalReduction></actuator>
+  </transmission>
+  <joint name="elbow_flex" type="revolute">
+    <origin xyz="-0.11257 -0.028 2.46331e-16" rpy="-1.22818e-15 5.75928e-16 1.5708"/>
+    <parent link="$(arg arm_prefix)_upper_arm_link"/>
+    <child link="$(arg arm_prefix)_lower_arm_link"/>
+    <axis xyz="0 0 1"/>
+    <limit effort="10" velocity="10" lower="-1.653" upper="1.654"/>
+  </joint>
+  <transmission name="elbow_flex_trans">
+    <type>transmission_interface/SimpleTransmission</type>
+    <joint name="elbow_flex"><hardwareInterface>hardware_interface/PositionJointInterface</hardwareInterface></joint>
+    <actuator name="motor3"><hardwareInterface>hardware_interface/PositionJointInterface</hardwareInterface><mechanicalReduction>1</mechanicalReduction></actuator>
+  </transmission>
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
File: src/so101_description/urdf/so101_arm_with_control.urdf.xacro (robot description, xacro)
@@ -11,7 +11,9 @@
     <xacro:arg name="usb_port"                default="/dev/lerobot_follower" />
     <xacro:arg name="real_robot_joint_config"       default="" />
-    <xacro:arg name="arm_type"                default="follower" />
     <xacro:arg name="command"                default="true" />
     <xacro:arg name="gazebo_controllers_config" default="$(find so101_control)/config/so101_follower_controllers.yaml" />
+    <xacro:arg name="arm_prefix" default="follower" />
+    <!-- Prefix for all URDF link names: "follower_" or "leader_".
+         Keeps both arms' TF frames unique in the global tree. -->
     <!-- ros2_control hardware interface — skipped when moveit_status=true -->
     <xacro:if value="${'$(arg moveit_status)' == 'false'}">
@@ -26,13 +28,24 @@
         </xacro:if>
     </xacro:if>
-    <!-- World anchor: Gazebo merges a model's 'world' link with its world frame,
-         so the arm is fixed at its spawn position instead of falling under gravity.
-         For real hardware this just adds a zero-offset root frame to the TF chain. -->
-    <link name="world"/>
-    <joint name="world_joint" type="fixed">
-        <parent link="world"/>
-        <child link="base_link"/>
-        <origin xyz="0 0 0" rpy="0 0 0"/>
-    </joint>
+    <!-- World anchor.
+         Gazebo requires this link to be literally named "world" to anchor the model.
+         For real hardware / MoveIt, use the prefixed name so both arms' TF chains
+         are unique in the global tree without frame_prefix. -->
+    <xacro:if value="${'$(arg sim_mode)' == 'gazebo'}">
+        <link name="world"/>
+        <joint name="world_joint" type="fixed">
+            <parent link="world"/>
+            <child link="$(arg arm_prefix)_base_link"/>
+            <origin xyz="0 0 0" rpy="0 0 0"/>
+        </joint>
+    </xacro:if>
+    <xacro:unless value="${'$(arg sim_mode)' == 'gazebo'}">
+        <link name="$(arg arm_prefix)_world"/>
+        <joint name="world_joint" type="fixed">
+            <parent link="$(arg arm_prefix)_world"/>
+            <child link="$(arg arm_prefix)_base_link"/>
+            <origin xyz="0 0 0" rpy="0 0 0"/>
+        </joint>
+    </xacro:unless>
     <!-- Robot links and joints (base_link → jaw_link) -->
     <xacro:include filename="$(find so101_description)/urdf/robots/so101_arm.urdf.xacro" />

File: src/so101_moveit_config/config/so101_follower.urdf.xacro (robot description, xacro)
@@ -2,9 +2,11 @@
 <robot xmlns:xacro="http://www.ros.org/wiki/xacro" name="so101_follower">
     <xacro:arg name="initial_positions_file" default="initial_positions.yaml" />
+    <!-- arm_prefix: "follower" or "leader" — must match what bringup RSP uses -->
+    <xacro:arg name="arm_prefix" default="follower" />
     <!-- World anchor — mirrors so101_arm_with_control.urdf.xacro so MoveIt has a root frame -->
-    <link name="world"/>
+    <link name="$(arg arm_prefix)_world"/>
     <joint name="world_joint" type="fixed">
-        <parent link="world"/>
-        <child link="base_link"/>
+        <parent link="$(arg arm_prefix)_world"/>
+        <child link="$(arg arm_prefix)_base_link"/>
         <origin xyz="0 0 0" rpy="0 0 0"/>
     </joint>
