Commit message: remove the old moveit package and create new 5dof package. also remove servo pakage for now

File: src/so101_description/urdf/robots/5dof_so101_arm.urdf.xacro (robot description, xacro)
@@ -229,5 +229,5 @@
     <child link="$(arg arm_prefix)_shoulder_link"/>
     <axis xyz="0 0 1"/>
-    <limit effort="10" velocity="10" lower="-2.055" upper="2.058"/>
+    <limit effort="10.0" velocity="10.0" lower="-2.055" upper="2.058"/>
   </joint>
   <transmission name="shoulder_pan_trans">
@@ -241,5 +241,5 @@
     <child link="$(arg arm_prefix)_upper_arm_link"/>
     <axis xyz="0 0 1"/>
-    <limit effort="10" velocity="10" lower="-2.018" upper="2.018"/>
+    <limit effort="10.0" velocity="10.0" lower="-2.018" upper="2.018"/>
   </joint>
   <transmission name="shoulder_lift_trans">
@@ -253,5 +253,5 @@
     <child link="$(arg arm_prefix)_lower_arm_link"/>
     <axis xyz="0 0 1"/>
-    <limit effort="10" velocity="10" lower="-1.653" upper="1.654"/>
+    <limit effort="10.0" velocity="10.0" lower="-1.653" upper="1.654"/>
   </joint>
   <transmission name="elbow_flex_trans">
@@ -265,5 +265,5 @@
     <child link="$(arg arm_prefix)_wrist_link"/>
     <axis xyz="0 0 1"/>
-    <limit effort="10" velocity="10" lower="-1.786" upper="1.790"/>
+    <limit effort="10.0" velocity="10.0" lower="-1.786" upper="1.790"/>
   </joint>
   <transmission name="wrist_flex_trans">
@@ -277,5 +277,5 @@
     <child link="$(arg arm_prefix)_gripper_link"/>
     <axis xyz="0 0 1"/>
-    <limit effort="10" velocity="10" lower="-3.194" upper="4.120"/>
+    <limit effort="10.0" velocity="10.0" lower="-3.194" upper="4.120"/>
   </joint>
   <transmission name="wrist_roll_trans">
@@ -289,5 +289,5 @@
     <child link="$(arg arm_prefix)_jaw_link"/>
     <axis xyz="0 0 1"/>
-    <limit effort="10" velocity="10" lower="-0.174533" upper="1.74533"/>
+    <limit effort="10.0" velocity="10.0" lower="-0.174533" upper="1.74533"/>
   </joint>
   <transmission name="gripper_trans">
