Commit message: -refactor: axes correction in 6dof urdf; -feat: add graspnode package; -refactor: add a separate calibration package for 5dof and 6dof arms

File: src/so101_description/urdf/robots/6dof_so101_arm_fixed.urdf.xacro (robot description, xacro)
@@ -159,5 +159,11 @@
     <parent link="$(arg arm_prefix)_base_link"/>
     <child link="$(arg arm_prefix)_shoulder_link"/>
-    <axis xyz="0.008727 -0.0 0.999962"/>
+    <!-- Axis negated (+Z -> -Z). PROVEN, not guessed: the 5dof arm is known-good, and its
+         shoulder_pan really turns about -Z (its axis line reads "0 0 1", but its origin
+         rpy="-3.14159 0 1.5708" rolls the frame 180 deg, so local +Z points down). Upstream's
+         CAD zeroes this servo the other way. Matches the hardware report.
+         Whole vector negated, so the ~0.5 deg CAD tilt survives.
+         Limits untouched: they bound the servo value, which an axis flip does not change. -->
+    <axis xyz="-0.008727 0.0 -0.999962"/>
     <limit lower="-2.06" upper="2.01" effort="3.35" velocity="2.0"/>
     <dynamics damping="0.6" friction="0.052"/>
@@ -222,5 +228,10 @@
     <parent link="$(arg arm_prefix)_wrist_pitch_link"/>
     <child link="$(arg arm_prefix)_wrist_yaw_link"/>
-    <axis xyz="0.014193 -5e-05 0.999899"/>
+    <!-- Axis negated (+Z -> -Z). INFERRED, NOT PROVEN — the 5dof arm has no wrist_yaw, so there
+         is nothing to compare against. Flipped because it is a turntable joint like shoulder_pan,
+         which IS proven flipped, and both come from the same CAD convention.
+         This is the one axis here that rests on a guess. If it renders backwards, negate it back
+         and nothing else needs to move. -->
+    <axis xyz="-0.014193 5e-05 -0.999899"/>
     <limit effort="3.35" lower="-1.40" upper="1.32" velocity="2.0"/>
     <dynamics damping="0.6" friction="0.052"/>
@@ -235,5 +246,10 @@
     <parent link="$(arg arm_prefix)_wrist_yaw_link"/>
     <child link="$(arg arm_prefix)_wrist_roll_link"/>
-    <axis xyz="0.999922 -0.008805 -0.008802"/>
+    <!-- Axis negated (+X -> -X). PROVEN: the known-good 5dof wrist_roll really turns about +Y
+         (its origin rpy="1.5708 0 3.14159" chains to that), and once the 6dof's 90 deg base yaw
+         is removed, upstream's +X lands on -Y — the opposite. Matches the hardware report.
+         Whole vector negated, so the ~0.5 deg CAD tilt survives.
+         Limits untouched: they bound the servo value, which an axis flip does not change. -->
+    <axis xyz="-0.999922 0.008805 0.008802"/>
     <limit effort="3.35" lower="-3.08" upper="3.09" velocity="2.0"/>
     <dynamics damping="0.6" friction="0.052"/>
@@ -252,4 +268,11 @@
     <parent link="$(arg arm_prefix)_wrist_roll_link"/>
     <child link="$(arg arm_prefix)_left_jaw_link"/>
+    <!-- ponytail: axis deliberately NOT negated, unlike pan/yaw/roll. The 5dof cross-check that
+         proved those does not apply here: the 5dof gripper is REVOLUTE (jaw pivots), this one is
+         PRISMATIC (jaw slides). Different mechanism -> comparing the two axes proves nothing.
+         The old "gripper is opposite" hardware report is also unusable: it was made while the
+         units bug rendered radians as metres, so the jaw was flying open by 1.3 m.
+         Test it after position_scale (0.02) is confirmed: command the gripper open. If it closes,
+         negate this vector and right_jaw_slider's to match. Limits stay either way. -->
     <axis xyz="0.008881 0.999923 0.008649"/>
     <limit effort="100" lower="0.00" upper="0.026" velocity="100"/>

File: src/so101_description/urdf/so101_arm_with_control.urdf.xacro (robot description, xacro)
@@ -28,12 +28,31 @@
            - gazebo : arm sits on the table (0, 0.40, 0.97). 6 mesh needs -90 deg yaw.
            - else   : world origin (0,0,0) -> REAL ROBOT SAFE default.-->
+    <!-- The dof==6 yaw is not a table fact, it is a CAD frame-convention fact:
+         at zero joints the 5 tip runs down base -Y, the 6 tip down base +X.
+         The -90 realigns 6 onto the 5 convention, but ONLY in the gazebo branch,
+         so real_robot dof:=6 still gets yaw 0 -> sim and real disagree by 90 deg
+         in the world frame. Harmless while 6 is sim-only; world-frame code on the
+         real 6 arm (scene_localizer, apriltag_world_localizer) would aim 90 deg
+         off. Decide then: apply the yaw in both branches, or rotate base_link in
+         6dof_so101_arm.urdf.xacro so both arms share one convention and this
+         dof special-case can be deleted. Check with:
+             ros2 run tf2_ros tf2_echo world follower_base_link -->
+    <!-- Compare args as quoted strings: '$(arg dof)' == '6'.
+         A property holding "6" is coerced to int by xacro, so ${dof_val == '6'}
+         is int-vs-str and silently False. -->
     <xacro:property name="sim_mode_val" value="$(arg sim_mode)"/>
-    <xacro:property name="dof_val"      value="$(arg dof)"/>
     <xacro:if value="${sim_mode_val == 'gazebo'}">
-        <xacro:property name="base_xyz" value="0 0.40 0.97"/>
-        <xacro:if value="${dof_val == '6'}">
+        <!-- z differs by dof: table top is at 1.0. The 5 mesh sits 3 cm above its own
+             base_link (base_so101_v2 visual origin z=0.0301, rolled +90 so mesh-y maps to
+             world-z), so 0.97 lands its lowest metal at 1.0001 — resting on the table. The 6
+             mesh (base_link.stl) starts at its origin, no offset, so the SAME 0.97 buries it
+             3 cm underground and shoulder_pan drives the base sideways through solid table ->
+             joint frozen. Lift the 6 to 1.0 so its base bottom sits on the surface. -->
+        <xacro:if value="${'$(arg dof)' == '6'}">
+            <xacro:property name="base_xyz" value="0 0.40 1.0"/>
             <xacro:property name="base_rpy" value="0 0 -1.5708"/>
         </xacro:if>
-        <xacro:unless value="${dof_val == '6'}">
+        <xacro:unless value="${'$(arg dof)' == '6'}">
+            <xacro:property name="base_xyz" value="0 0.40 0.97"/>
             <xacro:property name="base_rpy" value="0 0 0"/>
         </xacro:unless>
@@ -55,5 +74,8 @@
     </xacro:if>
     <xacro:if value="${'$(arg dof)' == '6'}">
-        <xacro:include filename="$(find so101_description)/urdf/robots/6dof_so101_arm.urdf.xacro" />
+        <!-- _fixed = axis signs corrected to this arm's servo convention (pan/yaw/roll negated).
+             Swap back to 6dof_so101_arm.urdf.xacro to A/B the old behaviour. Delete the old file
+             once _fixed is confirmed on hardware. -->
+        <xacro:include filename="$(find so101_description)/urdf/robots/6dof_so101_arm_fixed.urdf.xacro" />
     </xacro:if>
 </robot>
