Commit message: feat: add the new moveit config for the modified urdf

File: src/so101_description/urdf/so101_arm_with_control.urdf.xacro (robot description, xacro)
@@ -1,9 +1,3 @@
 <?xml version='1.0' encoding='utf-8'?>
-<!-- Per-arm entry point for namespaced launches.
-     Load this once per arm under its own ROS namespace.
-     The launch file handles:
-       - frame_prefix (so TF frames become follower/base_link, leader/base_link, etc.)
-       - static transform from table_link to <ns>/base_link (physical placement)
-     Joint names stay plain (shoulder_pan, shoulder_lift, ...) — no prefix needed. -->
 <robot name="so101_arm" xmlns:xacro="http://www.ros.org/wiki/xacro">
     <xacro:arg name="sim_mode"                default="real_robot" />
@@ -28,24 +22,11 @@
         </xacro:if>
     </xacro:if>
-    <!-- World anchor.
-         Gazebo requires this link to be literally named "world" to anchor the model.
-         For real hardware / MoveIt, use the prefixed name so both arms' TF chains
-         are unique in the global tree without frame_prefix. -->
-    <xacro:if value="${'$(arg sim_mode)' == 'gazebo'}">
-        <link name="world"/>
-        <joint name="world_joint" type="fixed">
-            <parent link="world"/>
-            <child link="$(arg arm_prefix)_base_link"/>
-            <origin xyz="0 0 0" rpy="0 0 0"/>
-        </joint>
-    </xacro:if>
-    <xacro:unless value="${'$(arg sim_mode)' == 'gazebo'}">
-        <link name="$(arg arm_prefix)_world"/>
-        <joint name="world_joint" type="fixed">
-            <parent link="$(arg arm_prefix)_world"/>
-            <child link="$(arg arm_prefix)_base_link"/>
-            <origin xyz="0 0 0" rpy="0 0 0"/>
-        </joint>
-    </xacro:unless>
+    <!-- World anchor — shared root for all arms in the scene. -->
+    <link name="world"/>
+    <joint name="world_joint" type="fixed">
+        <parent link="world"/>
+        <child link="$(arg arm_prefix)_base_link"/>
+        <origin xyz="0 0 0" rpy="0 0 0"/>
+    </joint>
     <!-- Robot links and joints (base_link → jaw_link) -->
     <xacro:include filename="$(find so101_description)/urdf/robots/so101_arm.urdf.xacro" />

File: src/so101_moveit_config/config/so101_arm.ros2_control.xacro (robot description, xacro)
@@ -1,5 +1,5 @@
 <?xml version="1.0"?>
 <robot xmlns:xacro="http://www.ros.org/wiki/xacro">
-    <xacro:macro name="so101_follower_ros2_control" params="name initial_positions_file">
+    <xacro:macro name="so101_arm_ros2_control" params="name initial_positions_file">
         <xacro:property name="initial_positions" value="${load_yaml(initial_positions_file)['initial_positions']}"/>
         <ros2_control name="${name}" type="system">
@@ -13,4 +13,5 @@
                   <param name="initial_value">${initial_positions['shoulder_pan']}</param>
                 </state_interface>
+                <state_interface name="velocity"/>
             </joint>
             <joint name="shoulder_lift">
@@ -19,4 +20,5 @@
                   <param name="initial_value">${initial_positions['shoulder_lift']}</param>
                 </state_interface>
+                <state_interface name="velocity"/>
             </joint>
             <joint name="elbow_flex">
@@ -25,4 +27,5 @@
                   <param name="initial_value">${initial_positions['elbow_flex']}</param>
                 </state_interface>
+                <state_interface name="velocity"/>
             </joint>
             <joint name="wrist_flex">
@@ -31,4 +34,5 @@
                   <param name="initial_value">${initial_positions['wrist_flex']}</param>
                 </state_interface>
+                <state_interface name="velocity"/>
             </joint>
             <joint name="wrist_roll">
@@ -37,4 +41,5 @@
                   <param name="initial_value">${initial_positions['wrist_roll']}</param>
                 </state_interface>
+                <state_interface name="velocity"/>
             </joint>
             <joint name="gripper">
@@ -43,4 +48,5 @@
                   <param name="initial_value">${initial_positions['gripper']}</param>
                 </state_interface>
+                <state_interface name="velocity"/>
             </joint>
         </ros2_control>
