Commit message: workspace maintenance: rename packages, clean metadata, reorganise launch files
Packages renamed:
- so101_interfaces → project_interfaces (fixed internal msg cross-refs)
- so101_teleop → joy_teleop (generic name)
- s0101_moveit_5dof → so101_moveit_5dof (typo fix)
- so101_6dof_moveit_config → so101_moveit_6dof (naming consistency)
- vlm → vlm_perception

All packages:
- package.xml: version 0.1.0, Apache-2.0, maintainer fixed, test_depends removed
- CMakeLists: removed C++ compiler flags + BUILD_TESTING lint blocks
- README.md added to every package

so101_description:
- dof_type → dof, dof_5/dof_6 → 5/6 (across 20 files)
- legacy URDF moved to legacy/

oakd_camera:
- 3 launch files renamed (real, sim_rsp, sim_pointcloud)
- 4 legacy launch files moved to legacy/

scene_db:
- scene.db untracked from git
- *.db added to workspace .gitignore

moveit_commander:
- Empty __init__.py removed
- TODO.md added (6DOF support needed)

so101_bringup:
- 17 launch files renamed with consistent {env}_{who}_{ctrl}.launch.py pattern
- debug_moveit_config.py moved to legacy/
- All internal cross-references updated

src/Changes.md added — full session log with date 2026-07-01

Co-Authored-By: Claude Sonnet 4.6 <noreply@anthropic.com>

File: src/so101_description/urdf/so101_arm_with_control.urdf.xacro (robot description, xacro)
@@ -8,5 +8,5 @@
     <xacro:arg name="gazebo_controllers_config" default="" />
     <xacro:arg name="arm_prefix" default="follower" />
-    <xacro:arg name="dof_type"   default="dof_5" />
+    <xacro:arg name="dof"   default="5" />
     <!-- Prefix for all URDF link names: "follower_" or "leader_".
          Keeps both arms' TF frames unique in the global tree. -->
@@ -25,15 +25,15 @@
     <!-- ============ ARM WORLD PLACEMENT — SINGLE SOURCE OF TRUTH ============
          world_joint = where the arm base sits in the world.
-         Chosen automatically by sim_mode (and dof_type for the yaw).
-           - gazebo : arm sits on the table (0, 0.40, 0.97). dof_6 mesh needs -90 deg yaw.
+         Chosen automatically by sim_mode (and dof for the yaw).
+           - gazebo : arm sits on the table (0, 0.40, 0.97). 6 mesh needs -90 deg yaw.
            - else   : world origin (0,0,0) -> REAL ROBOT SAFE default.-->
     <xacro:property name="sim_mode_val" value="$(arg sim_mode)"/>
-    <xacro:property name="dof_val"      value="$(arg dof_type)"/>
+    <xacro:property name="dof_val"      value="$(arg dof)"/>
     <xacro:if value="${sim_mode_val == 'gazebo'}">
         <xacro:property name="base_xyz" value="0 0.40 0.97"/>
-        <xacro:if value="${dof_val == 'dof_6'}">
+        <xacro:if value="${dof_val == '6'}">
             <xacro:property name="base_rpy" value="0 0 -1.5708"/>
         </xacro:if>
-        <xacro:unless value="${dof_val == 'dof_6'}">
+        <xacro:unless value="${dof_val == '6'}">
             <xacro:property name="base_rpy" value="0 0 0"/>
         </xacro:unless>
@@ -51,8 +51,8 @@
     </joint>
     <!-- Robot links and joints (base_link → jaw_link) -->
-    <xacro:if value="${'$(arg dof_type)' == 'dof_5'}">
+    <xacro:if value="${'$(arg dof)' == '5'}">
         <xacro:include filename="$(find so101_description)/urdf/robots/5dof_so101_arm.urdf.xacro" />
     </xacro:if>
-    <xacro:if value="${'$(arg dof_type)' == 'dof_6'}">
+    <xacro:if value="${'$(arg dof)' == '6'}">
         <xacro:include filename="$(find so101_description)/urdf/robots/6dof_so101_arm.urdf.xacro" />
     </xacro:if>
