Commit message: add new 6dof arm. change old arm to 5dof arm

File: src/so101_description/legacy/so101_follower.urdf (robot description, URDF)
Before this commit: robot so101_follower, 7 links, 6 joints
Links:
- link base_link: geometry collision mesh filename=package://so101_description/5dof_meshes/base_motor_holder_s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; collision mesh filename=package://so101_description/5dof_meshes/base_so101_v2.stl
- link gripper_link: geometry collision mesh filename=package://so101_description/5dof_meshes/sts3215_03a_v1.stl; collision mesh filename=package://so101_description/5dof_meshes/wrist_roll_follower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
- link jaw_link: geometry collision mesh filename=package://so101_description/5dof_meshes/moving_jaw_so101_v1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; visual mesh filename=package://so101_description/5dof_meshes/moving_jaw_so101_v1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
- link lower_arm_link: geometry collision mesh filename=package://so101_description/5dof_meshes/motor_holder_so101_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; collision mesh filename=package://so101_description/5dof_meshes/sts3215_03a_v1.stl
- link shoulder_link: geometry collision mesh filename=package://so101_description/5dof_meshes/motor_holder_so101_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; collision mesh filename=package://so101_description/5dof_meshes/rotation_pitch_so10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
- link upper_arm_link: geometry collision mesh filename=package://so101_description/5dof_meshes/sts3215_03a_v1.stl; collision mesh filename=package://so101_description/5dof_meshes/upper_arm_so101_v1.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
- link wrist_link: geometry collision mesh filename=package://so101_description/5dof_meshes/sts3215_03a_no_horn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; collision mesh filename=package://so101_description/5dof_meshes/wrist_roll_pitch_so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

File: src/so101_description/urdf/robots/5dof_so101_arm.urdf.xacro (robot description, xacro)
@@ -23,37 +23,37 @@
     <visual>
       <origin xyz="0.0206915 0.0221255 0.0300817" rpy="1.5708 -1.23909e-16 2.33147e-15"/>
-      <geometry><mesh filename="package://so101_description/meshes/base_motor_holder_so101_v1.stl"/></geometry>
+      <geometry><mesh filename="package://so101_description/5dof_meshes/base_motor_holder_so101_v1.stl"/></geometry>
       <material name="3d_printed"/>
     </visual>
     <collision>
       <origin xyz="0.0206915 0.0221255 0.0300817" rpy="1.5708 -1.23909e-16 2.33147e-15"/>
-      <geometry><mesh filename="package://so101_description/meshes/base_motor_holder_so101_v1.stl"/></geometry>
+      <geometry><mesh filename="package://so101_description/5dof_meshes/base_motor_holder_so101_v1.stl"/></geometry>
     </collision>
     <visual>
       <origin xyz="0.0207909 0.0221255 0.0300817" rpy="1.5708 -0 0"/>
-      <geometry><mesh filename="package://so101_description/meshes/base_so101_v2.stl"/></geometry>
+      <geometry><mesh filename="package://so101_description/5dof_meshes/base_so101_v2.stl"/></geometry>
       <material name="3d_printed"/>
     </visual>
     <collision>
       <origin xyz="0.0207909 0.0221255 0.0300817" rpy="1.5708 -0 0"/>
-      <geometry><mesh filename="package://so101_description/meshes/base_so101_v2.stl"/></geometry>
+      <geometry><mesh filename="package://so101_description/5dof_meshes/base_so101_v2.stl"/></geometry>
     </collision>
     <visual>
       <origin xyz="0.0207909 -0.0105745 0.0761817" rpy="-2.20282e-15 2.77556e-17 -1.5708"/>
-      <geometry><mesh filename="package://so101_description/meshes/sts3215_03a_v1.stl"/></geometry>
+      <geometry><mesh filename="package://so101_description/5dof_meshes/sts3215_03a_v1.stl"/></geometry>
       <material name="sts3215"/>
     </visual>
     <collision>
       <origin xyz="0.0207909 -0.0105745 0.0761817" rpy="-2.20282e-15 2.77556e-17 -1.5708"/>
-      <geometry><mesh filename="package://so101_description/meshes/sts3215_03a_v1.stl"/></geometry>
+      <geometry><mesh filename="package://so101_description/5dof_meshes/sts3215_03a_v1.stl"/></geometry>
     </collision>
     <visual>
       <origin xyz="0.0205915 0.0467435 0.0798817" rpy="1.5708 -1.21716e-14 2.33147e-15"/>
-      <geometry><mesh filename="package://so101_description/meshes/waveshare_mounting_plate_so101_v2.stl"/></geometry>
+      <geometry><mesh filename="package://so101_description/5dof_meshes/waveshare_mounting_plate_so101_v2.stl"/></geometry>
       <material name="3d_printed"/>
     </visual>
     <collision>
       <origin xyz="0.0205915 0.0467435 0.0798817" rpy="1.5708 -1.21716e-14 2.33147e-15"/>
-      <geometry><mesh filename="package://so101_description/meshes/waveshare_mounting_plate_so101_v2.stl"/></geometry>
+      <geometry><mesh filename="package://so101_description/5dof_meshes/waveshare_mounting_plate_so101_v2.stl"/></geometry>
     </collision>
   </link>
@@ -67,28 +67,28 @@
     <visual>
       <origin xyz="-0.0303992 0.000422241 -0.0417" rpy="1.5708 1.5708 0"/>
-      <geometry><mesh filename="package://so101_description/meshes/sts3215_03a_v1.stl"/></geometry>
+      <geometry><mesh filename="package://so101_description/5dof_meshes/sts3215_03a_v1.stl"/></geometry>
       <material name="sts3215"/>
     </visual>
     <collision>
       <origin xyz="-0.0303992 0.000422241 -0.0417" rpy="1.5708 1.5708 0"/>
-      <geometry><mesh filename="package://so101_description/meshes/sts3215_03a_v1.stl"/></geometry>
+      <geometry><mesh filename="package://so101_description/5dof_meshes/sts3215_03a_v1.stl"/></geometry>
     </collision>
     <visual>
       <origin xyz="-0.0675992 -0.000177759 0.0158499" rpy="1.5708 -1.5708 0"/>
-      <geometry><mesh filename="package://so101_description/meshes/motor_holder_so101_base_v1.stl"/></geometry>
+      <geometry><mesh filename="package://so101_description/5dof_meshes/motor_holder_so101_base_v1.stl"/></geometry>
       <material name="3d_printed"/>
     </visual>
     <collision>
       <origin xyz="-0.0675992 -0.000177759 0.0158499" rpy="1.5708 -1.5708 0"/>
-      <geometry><mesh filename="package://so101_description/meshes/motor_holder_so101_base_v1.stl"/></geometry>
+      <geometry><mesh filename="package://so101_description/5dof_meshes/motor_holder_so101_base_v1.stl"/></geometry>
     </collision>
     <visual>
       <origin xyz="0.0122008 2.22413e-05 0.0464" rpy="-1.5708 -0 0"/>
-      <geometry><mesh filename="package://so101_description/meshes/rotation_pitch_so101_v1.stl"/></geometry>
+      <geometry><mesh filename="package://so101_description/5dof_meshes/rotation_pitch_so101_v1.stl"/></geometry>
       <material name="3d_printed"/>
     </visual>
     <collision>
       <origin xyz="0.0122008 2.22413e-05 0.0464" rpy="-1.5708 -0 0"/>
-      <geometry><mesh filename="package://so101_description/meshes/rotation_pitch_so101_v1.stl"/></geometry>
+      <geometry><mesh filename="package://so101_description/5dof_meshes/rotation_pitch_so101_v1.stl"/></geometry>
     </collision>
   </link>
@@ -102,19 +102,19 @@
     <visual>
       <origin xyz="-0.11257 -0.0155 0.0187" rpy="-3.14159 -6.8695e-16 -1.5708"/>
-      <geometry><mesh filename="package://so101_description/meshes/sts3215_03a_v1.stl"/></geometry>
+      <geometry><mesh filename="package://so101_description/5dof_meshes/sts3215_03a_v1.stl"/></geometry>
       <material name="sts3215"/>
     </visual>
     <collision>
       <origin xyz="-0.11257 -0.0155 0.0187" rpy="-3.14159 -6.8695e-16 -1.5708"/>
-      <geometry><mesh filename="package://so101_description/meshes/sts3215_03a_v1.stl"/></geometry>
+      <geometry><mesh filename="package://so101_description/5dof_meshes/sts3215_03a_v1.stl"/></geometry>
     </collision>
     <visual>
       <origin xyz="-0.065085 0.012 0.0182" rpy="3.14159 -9.35612e-32 0"/>
-      <geometry><mesh filename="package://so101_description/meshes/upper_arm_so101_v1.stl"/></geometry>
+      <geometry><mesh filename="package://so101_description/5dof_meshes/upper_arm_so101_v1.stl"/></geometry>
       <material name="3d_printed"/>
     </visual>
     <collision>
       <origin xyz="-0.065085 0.012 0.0182" rpy="3.14159 -9.35612e-32 0"/>
-      <geometry><mesh filename="package://so101_description/meshes/upper_arm_so101_v1.stl"/></geometry>
+      <geometry><mesh filename="package://so101_description/5dof_meshes/upper_arm_so101_v1.stl"/></geometry>
     </collision>
   </link>
@@ -128,28 +128,28 @@
     <visual>
       <origin xyz="-0.0648499 -0.032 0.0182" rpy="-3.14159 -0 3.9443e-31"/>
-      <geometry><mesh filename="package://so101_description/meshes/under_arm_so101_v1.stl"/></geometry>
+      <geometry><mesh filename="package://so101_description/5dof_meshes/under_arm_so101_v1.stl"/></geometry>
       <material name="3d_printed"/>
     </visual>
     <collision>
       <origin xyz="-0.0648499 -0.032 0.0182" rpy="-3.14159 -0 3.9443e-31"/>
-      <geometry><mesh filename="package://so101_description/meshes/under_arm_so101_v1.stl"/></geometry>
+      <geometry><mesh filename="package://so101_description/5dof_meshes/under_arm_so101_v1.stl"/></geometry>
     </collision>
     <visual>
       <origin xyz="-0.0648499 -0.032 0.018" rpy="-3.14159 4.73317e-30 7.88861e-31"/>
-      <geometry><mesh filename="package://so101_description/meshes/motor_holder_so101_wrist_v1.stl"/></geometry>
+      <geometry><mesh filename="package://so101_description/5dof_meshes/motor_holder_so101_wrist_v1.stl"/></geometry>
       <material name="3d_printed"/>
     </visual>
     <collision>
       <origin xyz="-0.0648499 -0.032 0.018" rpy="-3.14159 4.73317e-30 7.88861e-31"/>
-      <geometry><mesh filename="package://so101_description/meshes/motor_holder_so101_wrist_v1.stl"/></geometry>
+      <geometry><mesh filename="package://so101_description/5dof_meshes/motor_holder_so101_wrist_v1.stl"/></geometry>
     </collision>
     <visual>
       <origin xyz="-0.1224 0.0052 0.0187" rpy="-3.14159 -3.58047e-15 -3.14159"/>
-      <geometry><mesh filename="package://so101_description/meshes/sts3215_03a_v1.stl"/></geometry>
+      <geometry><mesh filename="package://so101_description/5dof_meshes/sts3215_03a_v1.stl"/></geometry>
       <material name="sts3215"/>
     </visual>
     <collision>
       <origin xyz="-0.1224 0.0052 0.0187" rpy="-3.14159 -3.58047e-15 -3.14159"/>
-      <geometry><mesh filename="package://so101_description/meshes/sts3215_03a_v1.stl"/></geometry>
+      <geometry><mesh filename="package://so101_description/5dof_meshes/sts3215_03a_v1.stl"/></geometry>
     </collision>
   </link>
@@ -163,19 +163,19 @@
     <visual>
       <origin xyz="5.55112e-17 -0.0424 0.0306" rpy="1.5708 1.5708 0"/>
-      <geometry><mesh filename="package://so101_description/meshes/sts3215_03a_no_horn_v1.stl"/></geometry>
+      <geometry><mesh filename="package://so101_description/5dof_meshes/sts3215_03a_no_horn_v1.stl"/></geometry>
       <material name="sts3215"/>
     </visual>
     <collision>
       <origin xyz="5.55112e-17 -0.0424 0.0306" rpy="1.5708 1.5708 0"/>
-      <geometry><mesh filename="package://so101_description/meshes/sts3215_03a_no_horn_v1.stl"/></geometry>
+      <geometry><mesh filename="package://so101_description/5dof_meshes/sts3215_03a_no_horn_v1.stl"/></geometry>
     </collision>
     <visual>
       <origin xyz="0 -0.028 0.0181" rpy="-1.5708 -1.5708 0"/>
-      <geometry><mesh filename="package://so101_description/meshes/wrist_roll_pitch_so101_v2.stl"/></geometry>
+      <geometry><mesh filename="package://so101_description/5dof_meshes/wrist_roll_pitch_so101_v2.stl"/></geometry>
       <material name="3d_printed"/>
     </visual>
     <collision>
       <origin xyz="0 -0.028 0.0181" rpy="-1.5708 -1.5708 0"/>
-      <geometry><mesh filename="package://so101_description/meshes/wrist_roll_pitch_so101_v2.stl"/></geometry>
+      <geometry><mesh filename="package://so101_description/5dof_meshes/wrist_roll_pitch_so101_v2.stl"/></geometry>
     </collision>
   </link>
@@ -189,19 +189,19 @@
     <visual>
       <origin xyz="0.0077 0.0001 -0.0234" rpy="-1.5708 -5.55112e-17 -1.38213e-14"/>
-      <geometry><mesh filename="package://so101_description/meshes/sts3215_03a_v1.stl"/></geometry>
+      <geometry><mesh filename="package://so101_description/5dof_meshes/sts3215_03a_v1.stl"/></geometry>
       <material name="sts3215"/>
     </visual>
     <collision>
       <origin xyz="0.0077 0.0001 -0.0234" rpy="-1.5708 -5.55112e-17 -1.38213e-14"/>
-      <geometry><mesh filename="package://so101_description/meshes/sts3215_03a_v1.stl"/></geometry>
+      <geometry><mesh filename="package://so101_description/5dof_meshes/sts3215_03a_v1.stl"/></geometry>
     </collision>
     <visual>
       <origin xyz="5.55112e-17 -0.000218214 0.000949706" rpy="-3.14159 -5.55112e-17 -9.17912e-24"/>
-      <geometry><mesh filename="package://so101_description/meshes/wrist_roll_follower_so101_v1_nocamera.stl"/></geometry>
+      <geometry><mesh filename="package://so101_description/5dof_meshes/wrist_roll_follower_so101_v1_nocamera.stl"/></geometry>
       <material name="3d_printed"/>
     </visual>
     <collision>
       <origin xyz="5.55112e-17 -0.000218214 0.000949706" rpy="-3.14159 -5.55112e-17 -9.17912e-24"/>
-      <geometry><mesh filename="package://so101_description/meshes/wrist_roll_follower_so101_v1_nocamera.stl"/></geometry>
+      <geometry><mesh filename="package://so101_description/5dof_meshes/wrist_roll_follower_so101_v1_nocamera.stl"/></geometry>
     </collision>
   </link>
@@ -215,10 +215,10 @@
     <visual>
       <origin xyz="-5.55112e-17 -1.94746e-17 0.0189" rpy="9.53145e-17 -4.66093e-24 0"/>
-      <geometry><mesh filename="package://so101_description/meshes/moving_jaw_so101_v1.stl"/></geometry>
+      <geometry><mesh filename="package://so101_description/5dof_meshes/moving_jaw_so101_v1.stl"/></geometry>
       <material name="3d_printed"/>
     </visual>
     <collision>
       <origin xyz="-5.55112e-17 -1.94746e-17 0.0189" rpy="9.53145e-17 -4.66093e-24 0"/>
-      <geometry><mesh filename="package://so101_description/meshes/moving_jaw_so101_v1.stl"/></geometry>
+      <geometry><mesh filename="package://so101_description/5dof_meshes/moving_jaw_so101_v1.stl"/></geometry>
     </collision>
   </link>

File: src/so101_description/urdf/so101_arm_with_control.urdf.xacro (robot description, xacro)
@@ -6,6 +6,7 @@
     <xacro:arg name="real_robot_joint_config"       default="" />
     <xacro:arg name="command"                default="true" />
-    <xacro:arg name="gazebo_controllers_config" default="$(find so101_control)/config/so101_follower_controllers.yaml" />
+    <xacro:arg name="gazebo_controllers_config" default="" />
     <xacro:arg name="arm_prefix" default="follower" />
+    <xacro:arg name="dof_type"   default="dof_5" />
     <!-- Prefix for all URDF link names: "follower_" or "leader_".
          Keeps both arms' TF frames unique in the global tree. -->
@@ -30,4 +31,9 @@
     </joint>
     <!-- Robot links and joints (base_link → jaw_link) -->
-    <xacro:include filename="$(find so101_description)/urdf/robots/so101_arm.urdf.xacro" />
+    <xacro:if value="${'$(arg dof_type)' == 'dof_5'}">
+        <xacro:include filename="$(find so101_description)/urdf/robots/5dof_so101_arm.urdf.xacro" />
+    </xacro:if>
+    <xacro:if value="${'$(arg dof_type)' == 'dof_6'}">
+        <xacro:include filename="$(find so101_description)/urdf/robots/6dof_so101_arm.urdf.xacro" />
+    </xacro:if>
 </robot>
