Commit message: add depth camera to the moveit 6dof package

File: src/oakd_camera/urdf/oakd_camera_sim.urdf.xacro (robot description, xacro)
@@ -90,4 +90,18 @@
           <far>4.0</far>
         </clip>
+        <!-- Force correct intrinsics so camera_info MATCHES the 640x480 image.
+             gz Ignition rgbd_camera otherwise publishes a default 320x240 K
+             (cx=160,cy=120) -> wrong deprojection -> shifted cloud.
+             fx = fy = width / (2*tan(hfov/2)) = 640 / (2*tan(1.25/2)) = 441.
+             cx = width/2 = 320,  cy = height/2 = 240. -->
+        <lens>
+          <intrinsics>
+            <fx>441.0</fx>
+            <fy>441.0</fy>
+            <cx>320.0</cx>
+            <cy>240.0</cy>
+            <s>0.0</s>
+          </intrinsics>
+        </lens>
         <optical_frame_id>oak_rgb_camera_optical_frame</optical_frame_id>
       </camera>

File: src/so101_description/urdf/so101_arm_with_control.urdf.xacro (robot description, xacro)
@@ -23,4 +23,24 @@
         </xacro:if>
     </xacro:if>
+    <!-- ============ ARM WORLD PLACEMENT — SINGLE SOURCE OF TRUTH ============
+         world_joint = where the arm base sits in the world.
+         Chosen automatically by sim_mode (and dof_type for the yaw).
+           - gazebo : arm sits on the table (0, 0.40, 0.97). dof_6 mesh needs -90 deg yaw.
+           - else   : world origin (0,0,0) -> REAL ROBOT SAFE default.-->
+    <xacro:property name="sim_mode_val" value="$(arg sim_mode)"/>
+    <xacro:property name="dof_val"      value="$(arg dof_type)"/>
+    <xacro:if value="${sim_mode_val == 'gazebo'}">
+        <xacro:property name="base_xyz" value="0 0.40 0.97"/>
+        <xacro:if value="${dof_val == 'dof_6'}">
+            <xacro:property name="base_rpy" value="0 0 -1.5708"/>
+        </xacro:if>
+        <xacro:unless value="${dof_val == 'dof_6'}">
+            <xacro:property name="base_rpy" value="0 0 0"/>
+        </xacro:unless>
+    </xacro:if>
+    <xacro:unless value="${sim_mode_val == 'gazebo'}">
+        <xacro:property name="base_xyz" value="0 0 0"/>
+        <xacro:property name="base_rpy" value="0 0 0"/>
+    </xacro:unless>
     <!-- World anchor — shared root for all arms in the scene. -->
     <link name="world"/>
@@ -28,5 +48,5 @@
         <parent link="world"/>
         <child link="$(arg arm_prefix)_base_link"/>
-        <origin xyz="0 0 0" rpy="0 0 0"/>
+        <origin xyz="${base_xyz}" rpy="${base_rpy}"/>
     </joint>
     <!-- Robot links and joints (base_link → jaw_link) -->
